File: kit/TurtlePico/TurtlePico.kicad_pcb (KiCad board)
At the start: 4 copper layers, 63.5 x 99.3 mm, 49 parts, among them J1 USB-C, J10 LMotor, J11 Servo, J12 FR_ESC, J13 RR_ESC, J14 FL_ESC, J15 RL_ESC, J17 Lipo_In, J18 FR_PW, J19 RR_PW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

Commit message: edit connection
Routing:
- net Net-(J1-DN1): track 37.5 -> 41.0 mm
- net Net-(J1-DP1): track 32.6 -> 34.9 mm
