File: kit/TurtlePico/v0.0/TurtlePico.kicad_pcb (KiCad board)
At the start: 4 copper layers, 63.5 x 99.3 mm, 49 parts, among them J1 USB-C, J10 LMotor, J11 Servo, J12 FR_ESC, J13 RR_ESC, J14 FL_ESC, J15 RL_ESC, J17 Lipo_In, J18 FR_PW, J19 RR_PW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

Commit message: change version
Other:
- board text added: "Turtle Pico v0.0"
- board text removed: "Turtle Pico v1"
Changed lines of the file:
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@@
   (gr_arc (start 118.11 139.7) (mid 115.415923 138.584077) (end 114.3 135.89)
     (stroke (width 0.1) (type default)) (layer "Edge.Cuts"))
-  (gr_text "Turtle Pico v1" (at 166.37 82.55) (layer "B.SilkS")
+  (gr_text "Turtle Pico v0.0" (at 165.1 82.55) (layer "B.SilkS")
     (effects (font (size 2 2) (thickness 0.3) bold) (justify bottom mirror))
   )
