File: board/minimal/Connector.kicad_sch (KiCad schematic)
At the start: 7 parts, among them J12 Debug, J13 9DoF, J14 Temperature, J15 UltraSonic, J16 OLED

Commit message: update PCB and edit schematic
Parts:
- J12: footprint (none) -> Connector_JST:JST_PH_B3B-PH-SM4-TB_1x03-1MP_P2.00mm_Vertical
Changed lines of the file:
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@@
       (effects (font (size 1.27 1.27)))
     )
-    (property "Footprint" "" (at 170.18 88.9 0)
+    (property "Footprint" "Connector_JST:JST_PH_B3B-PH-SM4-TB_1x03-1MP_P2.00mm_Vertical" (at 170.18 88.9 0)
       (effects (font (size 1.27 1.27)) hide)
     )
