File: board/minimal/Audio.kicad_sch (KiCad schematic)
At the start: 12 parts, among them J9 AudioJack3, U10 PCM5102A

Commit message: add Weather to Dashboard
Parts:
- C32, C33, C37, C38: footprint Capacitor_SMD:C_0603_1608Metric -> Capacitor_SMD:C_0201_0603Metric
Changed lines of the file:
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@@
       (effects (font (size 1.27 1.27)) (justify left))
     )
-    (property "Footprint" "Capacitor_SMD:C_0603_1608Metric" (at 131.7752 109.22 0)
+    (property "Footprint" "Capacitor_SMD:C_0201_0603Metric" (at 131.7752 109.22 0)
       (effects (font (size 1.27 1.27)) hide)
     )
@@
       (effects (font (size 1.27 1.27)) (justify left))
     )
-    (property "Footprint" "Capacitor_SMD:C_0603_1608Metric" (at 145.7452 106.68 0)
+    (property "Footprint" "Capacitor_SMD:C_0201_0603Metric" (at 145.7452 106.68 0)
       (effects (font (size 1.27 1.27)) hide)
     )
@@
       (effects (font (size 1.27 1.27)) (justify left))
     )
-    (property "Footprint" "Capacitor_SMD:C_0603_1608Metric" (at 140.6652 106.68 0)
+    (property "Footprint" "Capacitor_SMD:C_0201_0603Metric" (at 140.6652 106.68 0)
       (effects (font (size 1.27 1.27)) hide)
     )
@@
       (effects (font (size 1.27 1.27)) (justify left))
     )
-    (property "Footprint" "Capacitor_SMD:C_0603_1608Metric" (at 138.43 115.8748 0)
-      (effects (font (size 1.27 1.27)) hide)
-    )
+    (property "Footprint" "Capacitor_SMD:C_0201_0603Metric" (at 138.43 115.8748 0)
+      (effects (font (size 1.27 1.27)) hide)
+    )
