File: board/minimal/LED_Switch.kicad_sch (KiCad schematic)
At the start: 14 parts, among them J10 LED, J11 LED, Q5 2SC4213, Q6 2SC4213, SW3 SW_{R}, SW4 SW_{L}, SW5 SW_DIP_x03

Commit message: update PCB and edit schematic
Parts:
- D3, D4: footprint (none) -> LED_SMD:LED_0603_1608Metric
- RV1: footprint (none) -> Potentiometer_SMD:Potentiometer_ACP_CA6-VSMD_Vertical
- SW3, SW4: footprint (none) -> SW_SKRPACE010:SW_SKRPACE010
- SW5: footprint (none) -> Package_DIP:SMDIP-6_W7.62mm
Changed lines of the file:
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@@
       (effects (font (size 1.27 1.27)) (justify right))
     )
-    (property "Footprint" "" (at 168.91 116.84 0)
+    (property "Footprint" "Potentiometer_SMD:Potentiometer_ACP_CA6-VSMD_Vertical" (at 168.91 116.84 0)
       (effects (font (size 1.27 1.27)) hide)
     )
@@
       (effects (font (size 1.27 1.27)))
     )
-    (property "Footprint" "" (at 114.3 109.22 0)
+    (property "Footprint" "LED_SMD:LED_0603_1608Metric" (at 114.3 109.22 0)
       (effects (font (size 1.27 1.27)) hide)
     )
@@
       (effects (font (size 1.27 1.27)))
     )
-    (property "Footprint" "" (at 167.64 102.87 0)
+    (property "Footprint" "SW_SKRPACE010:SW_SKRPACE010" (at 167.64 102.87 0)
       (effects (font (size 1.27 1.27)) hide)
     )
@@
       (effects (font (size 1.27 1.27)))
     )
-    (property "Footprint" "" (at 198.12 111.76 0)
+    (property "Footprint" "Package_DIP:SMDIP-6_W7.62mm" (at 198.12 111.76 0)
       (effects (font (size 1.27 1.27)) hide)
     )
@@
       (effects (font (size 1.27 1.27)))
     )
-    (property "Footprint" "" (at 167.64 95.25 0)
+    (property "Footprint" "SW_SKRPACE010:SW_SKRPACE010" (at 167.64 95.25 0)
       (effects (font (size 1.27 1.27)) hide)
     )
@@
       (effects (font (size 1.27 1.27)))
     )
-    (property "Footprint" "" (at 133.35 106.68 0)
-      (effects (font (size 1.27 1.27)) hide)
-    )
+    (property "Footprint" "LED_SMD:LED_0603_1608Metric" (at 133.35 106.68 0)
+      (effects (font (size 1.27 1.27)) hide)
+    )

Commit message: add Weather to Dashboard
Parts:
- SW5: footprint Package_DIP:SMDIP-6_W7.62mm -> DS04254203BKSMT:DS04254203BKSMT
- renumbered Q5 to Q3, Q6 to Q4
Changed lines of the file:
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@@
   (symbol (lib_id "Transistor_BJT:2SC4213") (at 142.24 114.3 0) (unit 1)
     (in_bom yes) (on_board yes) (dnp no)
-    (property "Reference" "Q6" (at 146.685 114.3 0)
+    (property "Reference" "Q4" (at 146.685 114.3 0)
       (effects (font (size 1.27 1.27)) (justify left))
     )
@@
       (project "TurtlePico-Minimal"
         (path "/7af2d99d-e350-48e7-86b4-20911ea922f3/3559871a-0f23-4a86-a659-f5f50e9db57b"
-          (reference "Q6") (unit 1)
+          (reference "Q4") (unit 1)
         )
       )
@@
   (symbol (lib_id "Transistor_BJT:2SC4213") (at 124.46 114.3 0) (unit 1)
     (in_bom yes) (on_board yes) (dnp no)
-    (property "Reference" "Q5" (at 119.38 113.03 0)
+    (property "Reference" "Q3" (at 119.38 113.03 0)
       (effects (font (size 1.27 1.27)) (justify left))
     )
@@
       (project "TurtlePico-Minimal"
         (path "/7af2d99d-e350-48e7-86b4-20911ea922f3/3559871a-0f23-4a86-a659-f5f50e9db57b"
-          (reference "Q5") (unit 1)
+          (reference "Q3") (unit 1)
         )
       )
@@
       (effects (font (size 1.27 1.27)))
     )
-    (property "Footprint" "Package_DIP:SMDIP-6_W7.62mm" (at 198.12 111.76 0)
-      (effects (font (size 1.27 1.27)) hide)
-    )
+    (property "Footprint" "DS04254203BKSMT:DS04254203BKSMT" (at 198.12 111.76 0)
+      (effects (font (size 1.27 1.27)) hide)
+    )
