File: board/minimal/RP2040.kicad_sch (KiCad schematic)
At the start: 30 parts, among them SW1 SW_Bootsel, SW2 SW_RST, U1 W25Q128JVS, U2 AP63203WU, U3 RP2040, Y1 ABLS-12.000MHZ-B4-T

Commit message: update PCB and edit schematic
Parts:
- C1, C10, C11, C12, C13, C14, C15, C16, C17, C18, C2, C3, C4, C5, C6, C7, C8, C9, L1: footprint (none) -> Capacitor_SMD:C_0603_1608Metric
- R1: footprint (none) -> Package_TO_SOT_SMD:SOT-223
- R2, R3, R4, R5: footprint (none) -> Resistor_SMD:R_0603_1608Metric
- SW1, SW2: footprint (none) -> SW_SKRPACE010:SW_SKRPACE010
- Y1: footprint (none) -> ABLS-12_000MHZ-B4-T:ABLS
Changed lines of the file:
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@@
       (effects (font (size 1.27 1.27)) (justify left))
     )
-    (property "Footprint" "" (at 66.04 107.188 90)
+    (property "Footprint" "Resistor_SMD:R_0603_1608Metric" (at 66.04 107.188 90)
       (effects (font (size 1.27 1.27)) hide)
     )
@@
       (effects (font (size 1.27 1.27)) (justify left))
     )
-    (property "Footprint" "" (at 66.04 97.028 90)
+    (property "Footprint" "Resistor_SMD:R_0603_1608Metric" (at 66.04 97.028 90)
       (effects (font (size 1.27 1.27)) hide)
     )
@@
       (effects (font (size 1.27 1.27)) (justify left))
     )
-    (property "Footprint" "" (at 71.12 130.048 90)
+    (property "Footprint" "Resistor_SMD:R_0603_1608Metric" (at 71.12 130.048 90)
       (effects (font (size 1.27 1.27)) hide)
     )
@@
       (effects (font (size 1.27 1.27)) (justify left))
     )
-    (property "Footprint" "" (at 109.22 77.978 90)
+    (property "Footprint" "Package_TO_SOT_SMD:SOT-223" (at 109.22 77.978 90)
       (effects (font (size 1.27 1.27)) hide)
     )
@@
       (effects (font (size 1.27 1.27)) (justify left))
     )
-    (property "Footprint" "" (at 176.2252 62.23 0)
+    (property "Footprint" "Capacitor_SMD:C_0603_1608Metric" (at 176.2252 62.23 0)
       (effects (font (size 1.27 1.27)) hide)
     )
@@
       (effects (font (size 1.27 1.27)) (justify left))
     )
-    (property "Footprint" "" (at 171.1452 62.23 0)
+    (property "Footprint" "Capacitor_SMD:C_0603_1608Metric" (at 171.1452 62.23 0)
       (effects (font (size 1.27 1.27)) hide)
     )
@@
       (effects (font (size 1.27 1.27)) (justify left))
     )
-    (property "Footprint" "" (at 181.3052 62.23 0)
+    (property "Footprint" "Capacitor_SMD:C_0603_1608Metric" (at 181.3052 62.23 0)
       (effects (font (size 1.27 1.27)) hide)
     )
@@
       (effects (font (size 1.27 1.27)) (justify left))
     )
-    (property "Footprint" "" (at 186.3852 62.23 0)
+    (property "Footprint" "Capacitor_SMD:C_0603_1608Metric" (at 186.3852 62.23 0)
       (effects (font (size 1.27 1.27)) hide)
     )
@@
       (effects (font (size 1.27 1.27)) (justify left))
     )
-    (property "Footprint" "" (at 201.6252 110.49 0)
+    (property "Footprint" "Capacitor_SMD:C_0603_1608Metric" (at 201.6252 110.49 0)
       (effects (font (size 1.27 1.27)) hide)
     )
@@
       (effects (font (size 1.27 1.27)) (justify left))
     )
-    (property "Footprint" "" (at 191.4652 62.23 0)
+    (property "Footprint" "Capacitor_SMD:C_0603_1608Metric" (at 191.4652 62.23 0)
       (effects (font (size 1.27 1.27)) hide)
     )
@@
       (effects (font (size 1.27 1.27)) (justify left))
     )
-    (property "Footprint" "" (at 160.9852 62.23 0)
+    (property "Footprint" "Capacitor_SMD:C_0603_1608Metric" (at 160.9852 62.23 0)
       (effects (font (size 1.27 1.27)) hide)
     )
@@
       (effects (font (size 1.27 1.27)))
     )
-    (property "Footprint" "" (at 237.49 101.6 0)
+    (property "Footprint" "Capacitor_SMD:C_0603_1608Metric" (at 237.49 101.6 0)
       (effects (font (size 1.27 1.27)) hide)
     )
@@
       (effects (font (size 1.27 1.27)) (justify left))
     )
-    (property "Footprint" "" (at 158.75 61.2648 0)
+    (property "Footprint" "Capacitor_SMD:C_0603_1608Metric" (at 158.75 61.2648 0)
       (effects (font (size 1.27 1.27)) hide)
     )
@@
       (effects (font (size 1.27 1.27)))
     )
-    (property "Footprint" "" (at 76.2 90.17 0)
+    (property "Footprint" "SW_SKRPACE010:SW_SKRPACE010" (at 76.2 90.17 0)
       (effects (font (size 1.27 1.27)) hide)
     )
@@
       (effects (font (size 1.27 1.27)) (justify left))
     )
-    (property "Footprint" "" (at 63.5 119.6848 0)
+    (property "Footprint" "Capacitor_SMD:C_0603_1608Metric" (at 63.5 119.6848 0)
       (effects (font (size 1.27 1.27)) hide)
     )
@@
       (effects (font (size 1.27 1.27)) (justify left))
     )
-    (property "Footprint" "" (at 63.5 127.3048 0)
+    (property "Footprint" "Capacitor_SMD:C_0603_1608Metric" (at 63.5 127.3048 0)
       (effects (font (size 1.27 1.27)) hide)
     )
@@
       (effects (font (size 1.27 1.27)) (justify left))
     )
-    (property "Footprint" "" (at 242.2652 114.3 0)
+    (property "Footprint" "Capacitor_SMD:C_0603_1608Metric" (at 242.2652 114.3 0)
       (effects (font (size 1.27 1.27)) hide)
     )
@@
       (effects (font (size 1.27 1.27)) (justify left))
     )
-    (property "Footprint" "" (at 233.68 103.1748 0)
+    (property "Footprint" "Capacitor_SMD:C_0603_1608Metric" (at 233.68 103.1748 0)
       (effects (font (size 1.27 1.27)) hide)
     )
@@
       (effects (font (size 1.27 1.27)) (justify left))
     )
-    (property "Footprint" "" (at 237.1852 114.3 0)
+    (property "Footprint" "Capacitor_SMD:C_0603_1608Metric" (at 237.1852 114.3 0)
       (effects (font (size 1.27 1.27)) hide)
     )
@@
       (effects (font (size 1.27 1.27)))
     )
-    (property "Footprint" "" (at 76.2 100.33 0)
+    (property "Footprint" "SW_SKRPACE010:SW_SKRPACE010" (at 76.2 100.33 0)
       (effects (font (size 1.27 1.27)) hide)
     )
@@
       (effects (font (size 1.27 1.27)) (justify left))
     )
-    (property "Footprint" "" (at 129.2352 60.96 0)
+    (property "Footprint" "Capacitor_SMD:C_0603_1608Metric" (at 129.2352 60.96 0)
       (effects (font (size 1.27 1.27)) hide)
     )
@@
       (effects (font (size 1.27 1.27)) (justify left))
     )
-    (property "Footprint" "" (at 124.1552 60.96 0)
+    (property "Footprint" "Capacitor_SMD:C_0603_1608Metric" (at 124.1552 60.96 0)
       (effects (font (size 1.27 1.27)) hide)
     )
@@
       (effects (font (size 1.27 1.27)) (justify left))
     )
-    (property "Footprint" "" (at 166.0652 62.23 0)
+    (property "Footprint" "Capacitor_SMD:C_0603_1608Metric" (at 166.0652 62.23 0)
       (effects (font (size 1.27 1.27)) hide)
     )
@@
       (effects (font (size 1.27 1.27)) (justify left))
     )
-    (property "Footprint" "" (at 55.5752 66.04 0)
+    (property "Footprint" "Capacitor_SMD:C_0603_1608Metric" (at 55.5752 66.04 0)
       (effects (font (size 1.27 1.27)) hide)
     )
@@
       (effects (font (size 1.27 1.27)) (justify right))
     )
-    (property "Footprint" "" (at 66.04 124.46 0)
+    (property "Footprint" "ABLS-12_000MHZ-B4-T:ABLS" (at 66.04 124.46 0)
       (effects (font (size 1.27 1.27)) hide)
     )
@@
       (effects (font (size 1.27 1.27)) (justify left))
     )
-    (property "Footprint" "" (at 119.0752 60.96 0)
+    (property "Footprint" "Capacitor_SMD:C_0603_1608Metric" (at 119.0752 60.96 0)
       (effects (font (size 1.27 1.27)) hide)
     )
@@
       (effects (font (size 1.27 1.27)) (justify left))
     )
-    (property "Footprint" "" (at 109.22 80.518 90)
-      (effects (font (size 1.27 1.27)) hide)
-    )
+    (property "Footprint" "Resistor_SMD:R_0603_1608Metric" (at 109.22 80.518 90)
+      (effects (font (size 1.27 1.27)) hide)
+    )

Commit message: add Weather to Dashboard
Parts:
- C1, C10, C11, C12, C13, C17, C18, C2, C3, C4, C5, C6, C7, C8, C9: footprint Capacitor_SMD:C_0603_1608Metric -> Capacitor_SMD:C_0201_0603Metric
- C14: footprint Capacitor_SMD:C_0603_1608Metric -> Capacitor_SMD:C_1206_3216Metric
- C15, C16: footprint Capacitor_SMD:C_0603_1608Metric -> Capacitor_SMD:C_0402_1005Metric
- R1: footprint Package_TO_SOT_SMD:SOT-223 -> Resistor_SMD:R_0603_1608Metric
Changed lines of the file:
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@@
       (effects (font (size 1.27 1.27)) (justify left))
     )
-    (property "Footprint" "Package_TO_SOT_SMD:SOT-223" (at 109.22 77.978 90)
+    (property "Footprint" "Resistor_SMD:R_0603_1608Metric" (at 109.22 77.978 90)
       (effects (font (size 1.27 1.27)) hide)
     )
@@
       (effects (font (size 1.27 1.27)) (justify left))
     )
-    (property "Footprint" "Capacitor_SMD:C_0603_1608Metric" (at 176.2252 62.23 0)
+    (property "Footprint" "Capacitor_SMD:C_0201_0603Metric" (at 176.2252 62.23 0)
       (effects (font (size 1.27 1.27)) hide)
     )
@@
       (effects (font (size 1.27 1.27)) (justify left))
     )
-    (property "Footprint" "Capacitor_SMD:C_0603_1608Metric" (at 171.1452 62.23 0)
+    (property "Footprint" "Capacitor_SMD:C_0201_0603Metric" (at 171.1452 62.23 0)
       (effects (font (size 1.27 1.27)) hide)
     )
@@
       (effects (font (size 1.27 1.27)) (justify left))
     )
-    (property "Footprint" "Capacitor_SMD:C_0603_1608Metric" (at 181.3052 62.23 0)
+    (property "Footprint" "Capacitor_SMD:C_0201_0603Metric" (at 181.3052 62.23 0)
       (effects (font (size 1.27 1.27)) hide)
     )
@@
       (effects (font (size 1.27 1.27)) (justify left))
     )
-    (property "Footprint" "Capacitor_SMD:C_0603_1608Metric" (at 186.3852 62.23 0)
+    (property "Footprint" "Capacitor_SMD:C_0201_0603Metric" (at 186.3852 62.23 0)
       (effects (font (size 1.27 1.27)) hide)
     )
@@
       (effects (font (size 1.27 1.27)) (justify left))
     )
-    (property "Footprint" "Capacitor_SMD:C_0603_1608Metric" (at 201.6252 110.49 0)
+    (property "Footprint" "Capacitor_SMD:C_1206_3216Metric" (at 201.6252 110.49 0)
       (effects (font (size 1.27 1.27)) hide)
     )
@@
       (effects (font (size 1.27 1.27)) (justify left))
     )
-    (property "Footprint" "Capacitor_SMD:C_0603_1608Metric" (at 191.4652 62.23 0)
+    (property "Footprint" "Capacitor_SMD:C_0201_0603Metric" (at 191.4652 62.23 0)
       (effects (font (size 1.27 1.27)) hide)
     )
@@
       (effects (font (size 1.27 1.27)) (justify left))
     )
-    (property "Footprint" "Capacitor_SMD:C_0603_1608Metric" (at 160.9852 62.23 0)
+    (property "Footprint" "Capacitor_SMD:C_0201_0603Metric" (at 160.9852 62.23 0)
       (effects (font (size 1.27 1.27)) hide)
     )
@@
       (effects (font (size 1.27 1.27)) (justify left))
     )
-    (property "Footprint" "Capacitor_SMD:C_0603_1608Metric" (at 158.75 61.2648 0)
+    (property "Footprint" "Capacitor_SMD:C_0201_0603Metric" (at 158.75 61.2648 0)
       (effects (font (size 1.27 1.27)) hide)
     )
@@
       (effects (font (size 1.27 1.27)) (justify left))
     )
-    (property "Footprint" "Capacitor_SMD:C_0603_1608Metric" (at 63.5 119.6848 0)
+    (property "Footprint" "Capacitor_SMD:C_0201_0603Metric" (at 63.5 119.6848 0)
       (effects (font (size 1.27 1.27)) hide)
     )
@@
       (effects (font (size 1.27 1.27)) (justify left))
     )
-    (property "Footprint" "Capacitor_SMD:C_0603_1608Metric" (at 63.5 127.3048 0)
+    (property "Footprint" "Capacitor_SMD:C_0201_0603Metric" (at 63.5 127.3048 0)
       (effects (font (size 1.27 1.27)) hide)
     )
@@
       (effects (font (size 1.27 1.27)) (justify left))
     )
-    (property "Footprint" "Capacitor_SMD:C_0603_1608Metric" (at 242.2652 114.3 0)
+    (property "Footprint" "Capacitor_SMD:C_0402_1005Metric" (at 242.2652 114.3 0)
       (effects (font (size 1.27 1.27)) hide)
     )
@@
       (effects (font (size 1.27 1.27)) (justify left))
     )
-    (property "Footprint" "Capacitor_SMD:C_0603_1608Metric" (at 233.68 103.1748 0)
+    (property "Footprint" "Capacitor_SMD:C_0201_0603Metric" (at 233.68 103.1748 0)
       (effects (font (size 1.27 1.27)) hide)
     )
@@
       (effects (font (size 1.27 1.27)) (justify left))
     )
-    (property "Footprint" "Capacitor_SMD:C_0603_1608Metric" (at 237.1852 114.3 0)
+    (property "Footprint" "Capacitor_SMD:C_0402_1005Metric" (at 237.1852 114.3 0)
       (effects (font (size 1.27 1.27)) hide)
     )
@@
       (effects (font (size 1.27 1.27)) (justify left))
     )
-    (property "Footprint" "Capacitor_SMD:C_0603_1608Metric" (at 129.2352 60.96 0)
+    (property "Footprint" "Capacitor_SMD:C_0201_0603Metric" (at 129.2352 60.96 0)
       (effects (font (size 1.27 1.27)) hide)
     )
@@
       (effects (font (size 1.27 1.27)) (justify left))
     )
-    (property "Footprint" "Capacitor_SMD:C_0603_1608Metric" (at 124.1552 60.96 0)
+    (property "Footprint" "Capacitor_SMD:C_0201_0603Metric" (at 124.1552 60.96 0)
       (effects (font (size 1.27 1.27)) hide)
     )
@@
       (effects (font (size 1.27 1.27)) (justify left))
     )
-    (property "Footprint" "Capacitor_SMD:C_0603_1608Metric" (at 166.0652 62.23 0)
+    (property "Footprint" "Capacitor_SMD:C_0201_0603Metric" (at 166.0652 62.23 0)
       (effects (font (size 1.27 1.27)) hide)
     )
@@
       (effects (font (size 1.27 1.27)) (justify left))
     )
-    (property "Footprint" "Capacitor_SMD:C_0603_1608Metric" (at 55.5752 66.04 0)
+    (property "Footprint" "Capacitor_SMD:C_0201_0603Metric" (at 55.5752 66.04 0)
       (effects (font (size 1.27 1.27)) hide)
     )
@@
       (effects (font (size 1.27 1.27)) (justify left))
     )
-    (property "Footprint" "Capacitor_SMD:C_0603_1608Metric" (at 119.0752 60.96 0)
-      (effects (font (size 1.27 1.27)) hide)
-    )
+    (property "Footprint" "Capacitor_SMD:C_0201_0603Metric" (at 119.0752 60.96 0)
+      (effects (font (size 1.27 1.27)) hide)
+    )
