File: board/minimal/Sensor.kicad_sch (KiCad schematic)
At the start: 28 parts, among them Q3 PMOS, Q4 PMOS, U5 TLV73318PDBV, U6 PCA9306D, U7 ICM-20948, U8 BME280, U9 INA260

Commit message: update PCB and edit schematic
Parts:
- C23, C24, C25, C26, C27, C28, C29, C30, C31: footprint (none) -> Capacitor_SMD:C_0603_1608Metric
- JP1, JP2, JP3: footprint (none) -> Jumper:SolderJumper-2_P1.3mm_Open_RoundedPad1.0x1.5mm
- Q3, Q4: footprint (none) -> Package_TO_SOT_SMD:SOT-223
- R13, R14, R15, R16, R17, R18, R19, R20, R21: footprint (none) -> Resistor_SMD:R_0603_1608Metric
Changed lines of the file:
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@@
   (junction (at 210.82 125.73) (diameter 0) (color 0 0 0 0)
+  )
+  (junction (at 95.25 78.74) (diameter 0) (color 0 0 0 0)
   )
   (junction (at 90.17 81.28) (diameter 0) (color 0 0 0 0)
@@
     )
   )
+  (symbol (lib_id "power:PWR_FLAG") (at 95.25 78.74 0) (unit 1)
+    (in_bom yes) (on_board yes) (dnp no)
+    (property "Reference" "#FLG05" (at 95.25 76.835 0)
+      (effects (font (size 1.27 1.27)) hide)
+    )
+    (property "Value" "PWR_FLAG" (at 101.6 77.47 0)
+      (effects (font (size 1.27 1.27)))
+    )
+    (property "Footprint" "" (at 95.25 78.74 0)
+      (effects (font (size 1.27 1.27)) hide)
+    )
+    (property "Datasheet" "~" (at 95.25 78.74 0)
+      (effects (font (size 1.27 1.27)) hide)
+    )
+    (pin "1")
+    (instances
+      (project "TurtlePico-Minimal"
+        (path "/7af2d99d-e350-48e7-86b4-20911ea922f3/399e14dd-2b99-438e-9945-456c74135ff2"
+          (reference "#FLG05") (unit 1)
+        )
+      )
+    )
+  )
   (symbol (lib_id "Device:R") (at 120.65 81.28 0) (unit 1)
     (in_bom yes) (on_board yes) (dnp no)
@@
       (effects (font (size 1.27 1.27)) (justify left))
     )
-    (property "Footprint" "" (at 118.872 81.28 90)
+    (property "Footprint" "Resistor_SMD:R_0603_1608Metric" (at 118.872 81.28 90)
       (effects (font (size 1.27 1.27)) hide)
     )
@@
       (effects (font (size 1.27 1.27)) (justify left))
     )
-    (property "Footprint" "" (at 176.2252 80.01 0)
+    (property "Footprint" "Capacitor_SMD:C_0603_1608Metric" (at 176.2252 80.01 0)
       (effects (font (size 1.27 1.27)) hide)
     )
@@
       (effects (font (size 1.27 1.27)) (justify left))
     )
-    (property "Footprint" "" (at 172.4152 140.97 0)
+    (property "Footprint" "Capacitor_SMD:C_0603_1608Metric" (at 172.4152 140.97 0)
       (effects (font (size 1.27 1.27)) hide)
     )
@@
       (effects (font (size 1.27 1.27)))
     )
-    (property "Footprint" "" (at 220.98 121.92 0)
+    (property "Footprint" "Jumper:SolderJumper-2_P1.3mm_Open_RoundedPad1.0x1.5mm" (at 220.98 121.92 0)
       (effects (font (size 1.27 1.27)) hide)
     )
@@
       (effects (font (size 1.27 1.27)) (justify left))
     )
-    (property "Footprint" "" (at 168.6052 80.01 0)
+    (property "Footprint" "Capacitor_SMD:C_0603_1608Metric" (at 168.6052 80.01 0)
       (effects (font (size 1.27 1.27)) hide)
     )
@@
       (effects (font (size 1.27 1.27)) (justify left))
     )
-    (property "Footprint" "" (at 88.392 85.09 90)
+    (property "Footprint" "Resistor_SMD:R_0603_1608Metric" (at 88.392 85.09 90)
       (effects (font (size 1.27 1.27)) hide)
     )
@@
       (effects (font (size 1.27 1.27)) (justify left))
     )
-    (property "Footprint" "" (at 185.1152 113.03 0)
+    (property "Footprint" "Capacitor_SMD:C_0603_1608Metric" (at 185.1152 113.03 0)
       (effects (font (size 1.27 1.27)) hide)
     )
@@
       (effects (font (size 1.27 1.27)) (justify left))
     )
-    (property "Footprint" "" (at 192.7352 113.03 0)
+    (property "Footprint" "Capacitor_SMD:C_0603_1608Metric" (at 192.7352 113.03 0)
       (effects (font (size 1.27 1.27)) hide)
     )
@@
       (effects (font (size 1.27 1.27)) (justify left))
     )
-    (property "Footprint" "" (at 139.192 78.74 90)
+    (property "Footprint" "Resistor_SMD:R_0603_1608Metric" (at 139.192 78.74 90)
       (effects (font (size 1.27 1.27)) hide)
     )
@@
       (effects (font (size 1.27 1.27)) (justify left))
     )
-    (property "Footprint" "" (at 125.4252 138.43 0)
+    (property "Footprint" "Capacitor_SMD:C_0603_1608Metric" (at 125.4252 138.43 0)
       (effects (font (size 1.27 1.27)) hide)
     )
@@
       (effects (font (size 1.27 1.27)) (justify left))
     )
-    (property "Footprint" "" (at 223.012 97.79 90)
+    (property "Footprint" "Resistor_SMD:R_0603_1608Metric" (at 223.012 97.79 90)
       (effects (font (size 1.27 1.27)) hide)
     )
@@
       (effects (font (size 1.27 1.27)))
     )
-    (property "Footprint" "" (at 99.06 128.27 0)
+    (property "Footprint" "Package_TO_SOT_SMD:SOT-223" (at 99.06 128.27 0)
       (effects (font (size 1.27 1.27)) hide)
     )
@@
       (effects (font (size 1.27 1.27)) (justify left))
     )
-    (property "Footprint" "" (at 131.7752 67.31 0)
+    (property "Footprint" "Capacitor_SMD:C_0603_1608Metric" (at 131.7752 67.31 0)
       (effects (font (size 1.27 1.27)) hide)
     )
@@
       (effects (font (size 1.27 1.27)) (justify left))
     )
-    (property "Footprint" "" (at 94.488 85.09 90)
+    (property "Footprint" "Resistor_SMD:R_0603_1608Metric" (at 94.488 85.09 90)
       (effects (font (size 1.27 1.27)) hide)
     )
@@
       (effects (font (size 1.27 1.27)) (justify left))
     )
-    (property "Footprint" "" (at 106.172 134.62 90)
+    (property "Footprint" "Resistor_SMD:R_0603_1608Metric" (at 106.172 134.62 90)
       (effects (font (size 1.27 1.27)) hide)
     )
@@
       (effects (font (size 1.27 1.27)) (justify left))
     )
-    (property "Footprint" "" (at 167.3352 106.68 0)
+    (property "Footprint" "Capacitor_SMD:C_0603_1608Metric" (at 167.3352 106.68 0)
       (effects (font (size 1.27 1.27)) hide)
     )
@@
       (effects (font (size 1.27 1.27)))
     )
-    (property "Footprint" "" (at 133.35 140.97 0)
+    (property "Footprint" "Jumper:SolderJumper-2_P1.3mm_Open_RoundedPad1.0x1.5mm" (at 133.35 140.97 0)
       (effects (font (size 1.27 1.27)) hide)
     )
@@
       (effects (font (size 1.27 1.27)))
     )
-    (property "Footprint" "" (at 116.84 128.27 0)
+    (property "Footprint" "Package_TO_SOT_SMD:SOT-223" (at 116.84 128.27 0)
       (effects (font (size 1.27 1.27)) hide)
     )
@@
       (effects (font (size 1.27 1.27)) (justify left))
     )
-    (property "Footprint" "" (at 119.38 140.208 90)
+    (property "Footprint" "Resistor_SMD:R_0603_1608Metric" (at 119.38 140.208 90)
       (effects (font (size 1.27 1.27)) hide)
     )
@@
       (effects (font (size 1.27 1.27)) (justify left))
     )
-    (property "Footprint" "" (at 115.062 81.28 90)
+    (property "Footprint" "Resistor_SMD:R_0603_1608Metric" (at 115.062 81.28 90)
       (effects (font (size 1.27 1.27)) hide)
     )
@@
       (effects (font (size 1.27 1.27)) (justify left))
     )
-    (property "Footprint" "" (at 115.2652 67.31 0)
+    (property "Footprint" "Capacitor_SMD:C_0603_1608Metric" (at 115.2652 67.31 0)
       (effects (font (size 1.27 1.27)) hide)
     )
@@
       (effects (font (size 1.27 1.27)) (justify left))
     )
-    (property "Footprint" "" (at 84.582 85.09 90)
+    (property "Footprint" "Resistor_SMD:R_0603_1608Metric" (at 84.582 85.09 90)
       (effects (font (size 1.27 1.27)) hide)
     )
@@
       (effects (font (size 1.27 1.27)))
     )
-    (property "Footprint" "" (at 134.62 83.82 0)
-      (effects (font (size 1.27 1.27)) hide)
-    )
+    (property "Footprint" "Jumper:SolderJumper-2_P1.3mm_Open_RoundedPad1.0x1.5mm" (at 134.62 83.82 0)
+      (effects (font (size 1.27 1.27)) hide)
+    )

Commit message: add Weather to Dashboard
Parts:
- removed Q3, Q4: PMOS, Package_TO_SOT_SMD:SOT-223, symbol Simulation_SPICE:PMOS
- added Q2: DMP6050SSD, Package_SO:SOIC-8_3.9x4.9mm_P1.27mm, symbol Transistor_FET:DMP6050SSD
- C23, C24, C25, C26, C27, C28, C29, C30, C31: footprint Capacitor_SMD:C_0603_1608Metric -> Capacitor_SMD:C_0201_0603Metric
Connections:
- net PW_EN: now also Q2.2 (G1), Q2.4 (G2)
- net VBUS: now also Q2.7 (D1), Q2.8 (D1)
- net at C30.1, JP3.1 (A), U9.1 (IN+)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: now also Q2.5 (D2), Q2.6 (D2)
- net at R20.1: now also Q2.1 (S1), Q2.3 (S2)
