File: board/minimal/Storage.kicad_sch (KiCad schematic)
At the start: 1 part, among them J1 Micro_SD

Commit message: add Weather to Dashboard
Parts:
- J1: footprint Connector_Card:microSD_HC_Hirose_DM3AT-SF-PEJM5 -> Connector_Card:microSD_HC_Hirose_DM3D-SF
Changed lines of the file:
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@@
       (effects (font (size 1.27 1.27)))
     )
-    (property "Footprint" "Connector_Card:microSD_HC_Hirose_DM3AT-SF-PEJM5" (at 203.2 92.71 0)
+    (property "Footprint" "Connector_Card:microSD_HC_Hirose_DM3D-SF" (at 203.2 92.71 0)
       (effects (font (size 1.27 1.27)) hide)
     )
